File: XBEE/Baquela2/Xbee/Xbee.sch (KiCad schematic (older format))
At the start: 4 parts, among them J1 Conn_01x08_Female, J2 Conn_01x10_Female, J3 Conn_01x10_Female, J4 Conn_01x08_Female

Commit message: Ductos
Connections:
- net GND: now reaches J2.10 (Pin_10), J4.8 (Pin_8)
Changed lines of the file:
@@
 	5900 3650 5900 4000
 Wire Wire Line
-	5900 4000 4050 4000
+	5900 4000 4450 4000
 Wire Wire Line
 	4050 4000 4050 3750
@@
 NoConn ~ 3650 3550
 NoConn ~ 3650 3450
+$Comp
+L power:GND #PWR0101
+U 1 1 5EBBF0A9
+P 4450 4250
+F 0 "#PWR0101" H 4450 4000 50  0001 C CNN
+F 1 "GND" H 4455 4077 50  0000 C CNN
+F 2 "" H 4450 4250 50  0001 C CNN
+F 3 "" H 4450 4250 50  0001 C CNN
+	1    4450 4250
+	1    0    0    -1
+$EndComp
+Wire Wire Line
+	4450 4250 4450 4000
+Connection ~ 4450 4000
+Wire Wire Line
+	4450 4000 4050 4000
 $EndSCHEMATC
