File: XBEE/Baquela2/Xbee/Xbee.kicad_pcb (KiCad board)
At the start: 2 copper layers, 36 x 29 mm, 4 parts, among them J1 Conn_01x08_Female, J2 Conn_01x10_Female, J3 Conn_01x10_Female, J4 Conn_01x08_Female

Commit message: niksd
Parts:
- added J1: Conn_01x04_Female, TerminalBlock:TerminalBlock_Altech_AK300-4_P5.00mm, B.Cu at (25.6, 116.2)
- added J1: Conn_01x08_Female, Connector_PinSocket_2.54mm:PinSocket_1x08_P2.54mm_Vertical, F.Cu at (59.6, 217.2)
- added J1: Conn_01x08_Female, Connector_PinSocket_2.54mm:PinSocket_1x08_P2.54mm_Vertical, F.Cu at (59.6, 185.4)
- added J1: Conn_01x08_Female, Connector_PinSocket_2.54mm:PinSocket_1x08_P2.54mm_Vertical, F.Cu at (22.8, 247.7)
- added J1: Conn_01x08_Female, Connector_PinSocket_2.54mm:PinSocket_1x08_P2.54mm_Vertical, F.Cu at (22.8, 217.2)
- added J1: Conn_01x04_Female, TerminalBlock:TerminalBlock_Altech_AK300-4_P5.00mm, B.Cu at (137.4, 116.2)
- added J1: Conn_01x04_Female, TerminalBlock:TerminalBlock_Altech_AK300-4_P5.00mm, B.Cu at (81.5, 116.2)
- added J1: Conn_01x04_Female, TerminalBlock:TerminalBlock_Altech_AK300-4_P5.00mm, B.Cu at (109.4, 116.2)
- added J1: Conn_01x04_Female, TerminalBlock:TerminalBlock_Altech_AK300-4_P5.00mm, B.Cu at (53.6, 170.9)
- added J1: Conn_01x04_Female, TerminalBlock:TerminalBlock_Altech_AK300-4_P5.00mm, B.Cu at (53.6, 116.2)
- added J1: Conn_01x04_Female, TerminalBlock:TerminalBlock_Altech_AK300-4_P5.00mm, B.Cu at (81.5, 170.9)
- added J1: Conn_01x04_Female, TerminalBlock:TerminalBlock_Altech_AK300-4_P5.00mm, B.Cu at (25.6, 170.9)
- added J1: Conn_01x04_Female, TerminalBlock:TerminalBlock_Altech_AK300-4_P5.00mm, B.Cu at (109.4, 170.9)
- added J1: Conn_01x04_Female, TerminalBlock:TerminalBlock_Altech_AK300-4_P5.00mm, B.Cu at (137.4, 170.9)
- added J1: Conn_01x08_Female, Connector_PinSocket_2.54mm:PinSocket_1x08_P2.54mm_Vertical, F.Cu at (133.3, 247.7)
- added J1: Conn_01x08_Female, Connector_PinSocket_2.54mm:PinSocket_1x08_P2.54mm_Vertical, F.Cu at (133.3, 217.2)
- added J1: Conn_01x08_Female, Connector_PinSocket_2.54mm:PinSocket_1x08_P2.54mm_Vertical, F.Cu at (133.3, 185.4)
- added J1: Conn_01x08_Female, Connector_PinSocket_2.54mm:PinSocket_1x08_P2.54mm_Vertical, F.Cu at (96.5, 247.7)
- added J1: Conn_01x08_Female, Connector_PinSocket_2.54mm:PinSocket_1x08_P2.54mm_Vertical, F.Cu at (96.5, 217.2)
- added J1: Conn_01x08_Female, Connector_PinSocket_2.54mm:PinSocket_1x08_P2.54mm_Vertical, F.Cu at (96.5, 185.4)
- added J1: Conn_01x08_Female, Connector_PinSocket_2.54mm:PinSocket_1x08_P2.54mm_Vertical, F.Cu at (59.6, 247.7)
- added J2: Conn_01x10_Female, Connector_PinSocket_2.00mm:PinSocket_1x10_P2.00mm_Vertical, F.Cu at (138.3, 268.0)
- added J2: Conn_01x10_Female, Connector_PinSocket_2.00mm:PinSocket_1x10_P2.00mm_Vertical, F.Cu at (27.8, 268.0)
- added J2: Conn_01x10_Female, Connector_PinSocket_2.00mm:PinSocket_1x10_P2.00mm_Vertical, F.Cu at (27.8, 237.5)
- added J2: Conn_01x10_Female, Connector_PinSocket_2.00mm:PinSocket_1x10_P2.00mm_Vertical, F.Cu at (138.3, 237.5)
- added J2: Conn_01x10_Female, Connector_PinSocket_2.00mm:PinSocket_1x10_P2.00mm_Vertical, F.Cu at (138.3, 205.8)
- added J2: Conn_01x10_Female, Connector_PinSocket_2.00mm:PinSocket_1x10_P2.00mm_Vertical, F.Cu at (101.5, 268.0)
- added J2: Conn_01x10_Female, Connector_PinSocket_2.00mm:PinSocket_1x10_P2.00mm_Vertical, F.Cu at (101.5, 237.5)
- added J2: Conn_01x10_Female, Connector_PinSocket_2.00mm:PinSocket_1x10_P2.00mm_Vertical, F.Cu at (101.5, 205.8)
- added J2: Conn_01x10_Female, Connector_PinSocket_2.00mm:PinSocket_1x10_P2.00mm_Vertical, F.Cu at (64.6, 268.0)
- added J2: Conn_01x10_Female, Connector_PinSocket_2.00mm:PinSocket_1x10_P2.00mm_Vertical, F.Cu at (64.6, 237.5)
- added J2: Conn_01x10_Female, Connector_PinSocket_2.00mm:PinSocket_1x10_P2.00mm_Vertical, F.Cu at (64.6, 205.8)
- added J3: Conn_01x10_Female, Connector_PinSocket_2.00mm:PinSocket_1x10_P2.00mm_Vertical, F.Cu at (138.3, 246.0)
- added J3: Conn_01x10_Female, Connector_PinSocket_2.00mm:PinSocket_1x10_P2.00mm_Vertical, F.Cu at (27.8, 246.0)
- added J3: Conn_01x10_Female, Connector_PinSocket_2.00mm:PinSocket_1x10_P2.00mm_Vertical, F.Cu at (27.8, 215.5)
- added J3: Conn_01x10_Female, Connector_PinSocket_2.00mm:PinSocket_1x10_P2.00mm_Vertical, F.Cu at (138.3, 215.5)
- added J3: Conn_01x10_Female, Connector_PinSocket_2.00mm:PinSocket_1x10_P2.00mm_Vertical, F.Cu at (138.3, 183.8)
- added J3: Conn_01x10_Female, Connector_PinSocket_2.00mm:PinSocket_1x10_P2.00mm_Vertical, F.Cu at (101.5, 246.0)
- added J3: Conn_01x10_Female, Connector_PinSocket_2.00mm:PinSocket_1x10_P2.00mm_Vertical, F.Cu at (101.5, 215.5)
- added J3: Conn_01x10_Female, Connector_PinSocket_2.00mm:PinSocket_1x10_P2.00mm_Vertical, F.Cu at (101.5, 183.8)
- added J3: Conn_01x10_Female, Connector_PinSocket_2.00mm:PinSocket_1x10_P2.00mm_Vertical, F.Cu at (64.6, 246.0)
- added J3: Conn_01x10_Female, Connector_PinSocket_2.00mm:PinSocket_1x10_P2.00mm_Vertical, F.Cu at (64.6, 215.5)
- added J3: Conn_01x10_Female, Connector_PinSocket_2.00mm:PinSocket_1x10_P2.00mm_Vertical, F.Cu at (64.6, 183.8)
- added J4: Conn_01x08_Female, Connector_PinSocket_2.54mm:PinSocket_1x08_P2.54mm_Vertical, F.Cu at (161.3, 247.7)
- added J4: Conn_01x08_Female, Connector_PinSocket_2.54mm:PinSocket_1x08_P2.54mm_Vertical, F.Cu at (50.8, 247.7)
- added J4: Conn_01x08_Female, Connector_PinSocket_2.54mm:PinSocket_1x08_P2.54mm_Vertical, F.Cu at (50.8, 217.2)
- added J4: Conn_01x08_Female, Connector_PinSocket_2.54mm:PinSocket_1x08_P2.54mm_Vertical, F.Cu at (161.3, 217.2)
- added J4: Conn_01x08_Female, Connector_PinSocket_2.54mm:PinSocket_1x08_P2.54mm_Vertical, F.Cu at (161.3, 185.4)
- added J4: Conn_01x08_Female, Connector_PinSocket_2.54mm:PinSocket_1x08_P2.54mm_Vertical, F.Cu at (124.5, 247.7)
- added J4: Conn_01x08_Female, Connector_PinSocket_2.54mm:PinSocket_1x08_P2.54mm_Vertical, F.Cu at (124.5, 217.2)
- added J4: Conn_01x08_Female, Connector_PinSocket_2.54mm:PinSocket_1x08_P2.54mm_Vertical, F.Cu at (124.5, 185.4)
- added J4: Conn_01x08_Female, Connector_PinSocket_2.54mm:PinSocket_1x08_P2.54mm_Vertical, F.Cu at (87.6, 247.7)
- added J4: Conn_01x08_Female, Connector_PinSocket_2.54mm:PinSocket_1x08_P2.54mm_Vertical, F.Cu at (87.6, 217.2)
- added J4: Conn_01x08_Female, Connector_PinSocket_2.54mm:PinSocket_1x08_P2.54mm_Vertical, F.Cu at (87.6, 185.4)
- added R1: R, Resistor_THT:R_Axial_DIN0207_L6.3mm_D2.5mm_P10.16mm_Horizontal, B.Cu at (29.2, 105.4)
- added R1: R, Resistor_THT:R_Axial_DIN0207_L6.3mm_D2.5mm_P10.16mm_Horizontal, B.Cu at (113.0, 160.0)
- added R1: R, Resistor_THT:R_Axial_DIN0207_L6.3mm_D2.5mm_P10.16mm_Horizontal, B.Cu at (29.2, 160.0)
- added R1: R, Resistor_THT:R_Axial_DIN0207_L6.3mm_D2.5mm_P10.16mm_Horizontal, B.Cu at (57.1, 160.0)
- added R1: R, Resistor_THT:R_Axial_DIN0207_L6.3mm_D2.5mm_P10.16mm_Horizontal, B.Cu at (85.1, 105.4)
- added R1: R, Resistor_THT:R_Axial_DIN0207_L6.3mm_D2.5mm_P10.16mm_Horizontal, B.Cu at (113.0, 105.4)
- added R1: R, Resistor_THT:R_Axial_DIN0207_L6.3mm_D2.5mm_P10.16mm_Horizontal, B.Cu at (141.0, 105.4)
- added R1: R, Resistor_THT:R_Axial_DIN0207_L6.3mm_D2.5mm_P10.16mm_Horizontal, B.Cu at (141.0, 160.0)
- added R1: R, Resistor_THT:R_Axial_DIN0207_L6.3mm_D2.5mm_P10.16mm_Horizontal, B.Cu at (85.1, 160.0)
- added R1: R, Resistor_THT:R_Axial_DIN0207_L6.3mm_D2.5mm_P10.16mm_Horizontal, B.Cu at (57.1, 105.4)
- added R2: R, Resistor_THT:R_Axial_DIN0207_L6.3mm_D2.5mm_P10.16mm_Horizontal, B.Cu at (29.2, 101.6)
- added R2: R, Resistor_THT:R_Axial_DIN0207_L6.3mm_D2.5mm_P10.16mm_Horizontal, B.Cu at (85.1, 101.6)
- added R2: R, Resistor_THT:R_Axial_DIN0207_L6.3mm_D2.5mm_P10.16mm_Horizontal, B.Cu at (29.2, 156.2)
- added R2: R, Resistor_THT:R_Axial_DIN0207_L6.3mm_D2.5mm_P10.16mm_Horizontal, B.Cu at (57.1, 156.2)
- added R2: R, Resistor_THT:R_Axial_DIN0207_L6.3mm_D2.5mm_P10.16mm_Horizontal, B.Cu at (113.0, 101.6)
- added R2: R, Resistor_THT:R_Axial_DIN0207_L6.3mm_D2.5mm_P10.16mm_Horizontal, B.Cu at (141.0, 101.6)
- added R2: R, Resistor_THT:R_Axial_DIN0207_L6.3mm_D2.5mm_P10.16mm_Horizontal, B.Cu at (57.1, 101.6)
- added R2: R, Resistor_THT:R_Axial_DIN0207_L6.3mm_D2.5mm_P10.16mm_Horizontal, B.Cu at (113.0, 156.2)
- added R2: R, Resistor_THT:R_Axial_DIN0207_L6.3mm_D2.5mm_P10.16mm_Horizontal, B.Cu at (85.1, 156.2)
- added R2: R, Resistor_THT:R_Axial_DIN0207_L6.3mm_D2.5mm_P10.16mm_Horizontal, B.Cu at (141.0, 156.2)
- added U1: SensordePresion, Boards:SensorPresion, B.Cu at (35.6, 141.8)
- added U1: SensordePresion, Boards:SensorPresion, B.Cu at (147.4, 141.8)
- added U1: SensordePresion, Boards:SensorPresion, B.Cu at (35.6, 87.2)
- added U1: SensordePresion, Boards:SensorPresion, B.Cu at (91.5, 87.2)
- added U1: SensordePresion, Boards:SensorPresion, B.Cu at (119.4, 87.2)
- added U1: SensordePresion, Boards:SensorPresion, B.Cu at (147.4, 87.2)
- added U1: SensordePresion, Boards:SensorPresion, B.Cu at (63.6, 141.8)
- added U1: SensordePresion, Boards:SensorPresion, B.Cu at (119.4, 141.8)
- added U1: SensordePresion, Boards:SensorPresion, B.Cu at (63.6, 87.2)
- added U1: SensordePresion, Boards:SensorPresion, B.Cu at (91.5, 141.8)
- moved J1 166.3 mm to (22.8, 185.4)
- moved J2 166.3 mm to (27.8, 205.8)
- moved J3 166.3 mm to (27.8, 183.8)
- moved J4 166.3 mm to (50.8, 185.4)
Routing:
- net (no net): track 0.00 -> 3436.3 mm, vias 0 -> 20
- removed copper zone on B.Cu, net GND
Other:
- board size 36 x 29 mm -> 146.5 x 200.9 mm

Commit message: quien sabe
Parts:
- removed the J1 at (25.6, 116.2)
- removed the J1 at (59.6, 217.2)
- removed the J1 at (59.6, 185.4)
- removed the J1 at (22.8, 247.7)
- removed the J1 at (22.8, 217.2)
- removed the J1 at (137.4, 116.2)
- removed the J1 at (81.5, 116.2)
- removed the J1 at (109.4, 116.2)
- removed the J1 at (53.6, 170.9)
- removed the J1 at (53.6, 116.2)
- removed the J1 at (81.5, 170.9)
- removed the J1 at (25.6, 170.9)
- removed the J1 at (109.4, 170.9)
- removed the J1 at (137.4, 170.9)
- removed the J1 at (133.3, 247.7)
- removed the J1 at (133.3, 217.2)
- removed the J1 at (133.3, 185.4)
- removed the J1 at (96.5, 247.7)
- removed the J1 at (96.5, 217.2)
- removed the J1 at (96.5, 185.4)
- removed the J1 at (59.6, 247.7)
- removed the J2 at (138.3, 268.0)
- removed the J2 at (27.8, 268.0)
- removed the J2 at (27.8, 237.5)
- removed the J2 at (138.3, 237.5)
- removed the J2 at (138.3, 205.8)
- removed the J2 at (101.5, 268.0)
- removed the J2 at (101.5, 237.5)
- removed the J2 at (101.5, 205.8)
- removed the J2 at (64.6, 268.0)
- removed the J2 at (64.6, 237.5)
- removed the J2 at (64.6, 205.8)
- removed the J3 at (138.3, 246.0)
- removed the J3 at (27.8, 246.0)
- removed the J3 at (27.8, 215.5)
- removed the J3 at (138.3, 215.5)
- removed the J3 at (138.3, 183.8)
- removed the J3 at (101.5, 246.0)
- removed the J3 at (101.5, 215.5)
- removed the J3 at (101.5, 183.8)
- removed the J3 at (64.6, 246.0)
- removed the J3 at (64.6, 215.5)
- removed the J3 at (64.6, 183.8)
- removed the J4 at (161.3, 247.7)
- removed the J4 at (50.8, 247.7)
- removed the J4 at (50.8, 217.2)
- removed the J4 at (161.3, 217.2)
- removed the J4 at (161.3, 185.4)
- removed the J4 at (124.5, 247.7)
- removed the J4 at (124.5, 217.2)
- removed the J4 at (124.5, 185.4)
- removed the J4 at (87.6, 247.7)
- removed the J4 at (87.6, 217.2)
- removed the J4 at (87.6, 185.4)
- removed R1 (x10), R2 (x10): R, Resistor_THT:R_Axial_DIN0207_L6.3mm_D2.5mm_P10.16mm_Horizontal
- removed U1 (x10): SensordePresion, Boards:SensorPresion
- moved J1 115.9 mm to (107.9, 106.7)
- moved J2 115.9 mm to (112.9, 127.0)
- moved J3 115.9 mm to (112.9, 105.0)
- moved J4 115.9 mm to (135.9, 106.7)
Routing:
- net (no net): track 3436.3 -> 0.00 mm, vias 20 -> 0
Other:
- board size 146.5 x 200.9 mm -> 36 x 29 mm
