File: ESP8266_micro/Tarjeta/Covid/Covid.kicad_pcb (KiCad board)
At the start: 2 copper layers, 157.5 x 110.5 mm, 13 parts, among them U1 ESP32, U10 SOURCE, U2 LASER, U3 AMPLIFICADOR, U4 Trinket_M0, U5 JQ6500-16P, U6 L7805, U7 Boton_IR, U8 Boton_IR, U9 MLX90614

Commit message: arreglos en el codigo
Parts:
- removed REF**: ESD-Logo_13.2x12mm_SilkScreen, Symbol:ESD-Logo_13.2x12mm_SilkScreen
- added U11: Pantalla_SPI, Covid:Pantalla_spi, F.Cu at (132.1, 45.7)
Connections:
- U1 pad 12: Net-(U1-Pad12) -> TX_RX_AUDIO
- U1 pad 13: Net-(U1-Pad13) -> RX_TX_AUDIO
- U1 pad 23: Net-(U1-Pad23) -> CS
- U1 pad 24: Net-(U1-Pad24) -> RESET
- U1 pad 26: Net-(U1-Pad26) -> DC
- U1 pad 30: RX_TX_AUDIO -> SCK
- U1 pad 31: TX_RX_AUDIO -> MISO
- U1 pad 37: Net-(U1-Pad37) -> MOSI
Routing:
- net CS: track 0.00 -> 100.2 mm, vias 0 -> 1
- net RESET: track 0.00 -> 86.2 mm, vias 0 -> 1
- net DC: track 0.00 -> 81.6 mm, vias 0 -> 1
- net SCK: track 0.00 -> 69.3 mm, vias 0 -> 1
- net MOSI: track 0.00 -> 62.7 mm, vias 0 -> 1
- net TX_RX_AUDIO: track 21.8 -> 84.5 mm, vias 0 -> 1
- net RX_TX_AUDIO: track 21.8 -> 84.5 mm, vias 0 -> 1
- net MISO: track 0.00 -> 58.0 mm
- net VCC_3V: track 51.3 -> 105.8 mm
- net VCC_5V: track 185.3 -> 238.3 mm
- added copper zone on F.Cu, net GND

Commit message: pcb
Parts:
- removed C1, C2: CP, Covid:CAP_1uf
- added J1: Conn_01x04_Male, TerminalBlock_TE-Connectivity:TerminalBlock_TE_282834-4_1x04_P2.54mm_Horizontal, F.Cu at (119.4, 59.7)
- added J2: Conn_01x04_Male, TerminalBlock_TE-Connectivity:TerminalBlock_TE_282834-4_1x04_P2.54mm_Horizontal, F.Cu at (135.9, 59.7)
- added Q1: 2N2219, Package_TO_SOT_THT:TO-92L_Inline, F.Cu at (111.8, 125.7)
- added R1: R, Resistor_THT:R_Axial_DIN0309_L9.0mm_D3.2mm_P2.54mm_Vertical, F.Cu at (110.5, 118.1)
- added R2: R, Resistor_THT:R_Axial_DIN0309_L9.0mm_D3.2mm_P2.54mm_Vertical, F.Cu at (99.1, 53.3)
- added R3: R, Resistor_THT:R_Axial_DIN0309_L9.0mm_D3.2mm_P2.54mm_Vertical, F.Cu at (108.0, 38.1)
- added U12: LASER, Covid:LASER, F.Cu at (128.3, 139.7)
- added U13: MLX90614, TerminalBlock_TE-Connectivity:TerminalBlock_TE_282834-4_1x04_P2.54mm_Horizontal, F.Cu at (125.7, 45.7)
- U6: value L7805 -> Regulador; footprint Converter_DCDC:Converter_DCDC_muRata_OKI-78SR_Vertical -> Covid:Regulador
- moved U6 34.2 mm to (167.6, 124.5), turned to 180 degrees
- moved U10 26.9 mm to (160.0, 139.7)
Connections:
- U1 pad 12: TX_RX_AUDIO -> Net-(U1-Pad12)
- U1 pad 13: RX_TX_AUDIO -> Net-(U1-Pad13)
- U1 pad 16: Net-(U1-Pad16) -> TX_TAR_SON
- U1 pad 17: Net-(U1-Pad17) -> RX_TAR_SON
- U1 pad 30: SCK -> RX_SCK
- U1 pad 31: MISO -> TX_MISO
- U1 pad 8: Net-(U1-Pad8) -> SIRENA
Routing:
- net RX_TAR_SON: track 0.00 -> 153.8 mm
- net TX_TAR_SON: track 0.00 -> 130.7 mm, vias 0 -> 1
- net SIRENA: track 0.00 -> 76.5 mm
- net RX_SCK: track 0.00 -> 64.8 mm
- net TX_RX_AUDIO: track 84.5 -> 22.0 mm, vias 1 -> 0
- net SCK: track 69.3 -> 14.5 mm, vias 1 -> 0
- net RX_TX_AUDIO: track 84.5 -> 39.6 mm, vias 1 -> 0
- net TX_MISO: track 0.00 -> 40.5 mm
- net MISO: track 58.0 -> 22.2 mm
- net VCC_3V: track 105.8 -> 139.4 mm
- net VCC_5V: track 238.3 -> 269.8 mm, vias 0 -> 2
- net SCL: track 32.6 -> 61.9 mm
- net Net-(Q1-Pad3): track 0.00 -> 26.0 mm
- net SDA: track 39.8 -> 57.0 mm
- net AUDIO+: track 55.8 -> 68.9 mm
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